Commit message: Fixed collision geometry

File: tugbot_description/urdf/tugbot.urdf.xacro (robot description, xacro)
@@ -66,5 +66,5 @@
     </visual>
     <collision>
-      <origin xyz="0 0 0.03" rpy="0 0 0" />
+      <origin xyz="0 0 0.04" rpy="0 0 0" />
       <geometry>
         <box size="${base_x_size} ${base_y_size} ${base_z_size/2}"/>

Commit message: Final body collision params

File: tugbot_description/urdf/tugbot.urdf.xacro (robot description, xacro)
@@ -47,5 +47,5 @@
 	</xacro:macro>
   <!-- Base Size -->
-  <xacro:property name="base_x_size" value="0.42" />
+  <xacro:property name="base_x_size" value="0.44" />
   <xacro:property name="base_y_size" value="0.22" />
   <xacro:property name="base_z_size" value="0.17" />
@@ -66,5 +66,5 @@
     </visual>
     <collision>
-      <origin xyz="0 0 0.04" rpy="0 0 0" />
+      <origin xyz="0 0 0.035" rpy="0 0 0" />
       <geometry>
         <box size="${base_x_size} ${base_y_size} ${base_z_size/2}"/>

Commit message: Somewhat working simulation for driving around

File: tugbot_description/urdf/tugbot.urdf.xacro (robot description, xacro)
@@ -3,5 +3,5 @@
   <xacro:arg name="robot_namespace" default="/" />
   <xacro:property name="M_PI" value="3.14159"/>
-  <xacro:macro name="tugbot_wheel" params="wheel_prefix *joint_pose">
+  <xacro:macro name="tugbot_wheel" params="wheel_prefix left_wheel *joint_pose">
 		<link name="${wheel_prefix}_wheel_link">
 			<inertial>
@@ -11,5 +11,10 @@
 			</inertial>
 			<visual>
-				<origin xyz="0 0 0" rpy="0 0 ${M_PI/2}" />
+        <xacro:if value="${left_wheel}">
+				  <origin xyz="0 0 0" rpy="0 0 ${M_PI/2}" />
+        </xacro:if>
+        <xacro:unless value="${left_wheel}">
+				  <origin xyz="0 0 0" rpy="0 0 ${-M_PI/2}" />
+        </xacro:unless>
 				<geometry>
 					<mesh filename="package://tugbot_description/meshes/wheel.dae" />
@@ -72,9 +77,10 @@
     </collision>
   </link>
+    <!-- TODO: Work out actual inerias and mass-->
     <link name="inertial_link">
     <inertial>
-      <mass value="10.0" />
-      <origin xyz="-0.00065 -0.085 0.062" />
-      <inertia ixx="0.6022" ixy="-0.02364" ixz="-0.1197" iyy="1.7386" iyz="-0.001544" izz="2.0296" />
+      <mass value="1.0" />
+      <origin xyz="0 0 0" />
+      <inertia ixx="0.009375" ixy="0" ixz="0" iyy="0.009375" iyz="0" izz="0.009375" />
     </inertial>
   </link>
@@ -84,15 +90,15 @@
     <child link="inertial_link" />
   </joint>
-  <xacro:tugbot_wheel wheel_prefix="front_left">
+  <xacro:tugbot_wheel wheel_prefix="front_left" left_wheel="true">
     <origin xyz="${wheelbase/2} ${track/2} ${wheel_vertical_offset}" rpy="0 0 0" />
   </xacro:tugbot_wheel>
-  <xacro:tugbot_wheel wheel_prefix="front_right">
-    <origin xyz="${wheelbase/2} ${-track/2} ${wheel_vertical_offset}" rpy="0 0 ${M_PI}" />
+  <xacro:tugbot_wheel wheel_prefix="front_right" left_wheel="false">
+    <origin xyz="${wheelbase/2} ${-track/2} ${wheel_vertical_offset}" rpy="0 0 0" />
   </xacro:tugbot_wheel>
-  <xacro:tugbot_wheel wheel_prefix="rear_left">
+  <xacro:tugbot_wheel wheel_prefix="back_left" left_wheel="true">
     <origin xyz="${-wheelbase/2} ${track/2} ${wheel_vertical_offset}" rpy="0 0 0" />
   </xacro:tugbot_wheel>
-  <xacro:tugbot_wheel wheel_prefix="rear_right">
-    <origin xyz="${-wheelbase/2} ${-track/2} ${wheel_vertical_offset}" rpy="0 0 ${M_PI}" />
+  <xacro:tugbot_wheel wheel_prefix="back_right" left_wheel="false">
+    <origin xyz="${-wheelbase/2} ${-track/2} ${wheel_vertical_offset}" rpy="0 0 0" />
   </xacro:tugbot_wheel>
   <gazebo>

Commit message: Basic 2D slam

File: tugbot_description/urdf/tugbot.urdf.xacro (robot description, xacro)
@@ -6,7 +6,12 @@
 		<link name="${wheel_prefix}_wheel_link">
 			<inertial>
-				<mass value="2.637" />
-				<origin xyz="0 0 0" />
-				<inertia  ixx="0.02467" ixy="0" ixz="0" iyy="0.04411" iyz="0" izz="0.02467" />
+				<mass value="1.0" />
+				 <xacro:if value="${left_wheel}">
+				  <origin xyz="0 0.03 0" />
+        </xacro:if>
+        <xacro:unless value="${left_wheel}">
+				  <origin xyz="0 -0.03 0"/>
+        </xacro:unless>
+				<inertia  ixx="0.002467" ixy="0" ixz="0" iyy="0.004411" iyz="0" izz="0.002467" />
 			</inertial>
 			<visual>
@@ -22,5 +27,10 @@
 			</visual>
 			<collision>
-				<origin xyz="0 0.03 0" rpy="${M_PI/2} 0 0" />
+        <xacro:if value="${left_wheel}">
+				  <origin xyz="0 0.03 0" rpy="${M_PI/2} 0 0" />
+        </xacro:if>
+        <xacro:unless value="${left_wheel}">
+				  <origin xyz="0 -0.03 0" rpy="${M_PI/2} 0 0" />
+        </xacro:unless>
 				<geometry>
 					<cylinder length="${wheel_length}" radius="${wheel_radius}" />
@@ -82,5 +92,5 @@
       <mass value="1.0" />
       <origin xyz="0 0 0" />
-      <inertia ixx="0.009375" ixy="0" ixz="0" iyy="0.009375" iyz="0" izz="0.009375" />
+      <inertia ixx="0.010375" ixy="0" ixz="0" iyy="0.005375" iyz="0" izz="0.02375" />
     </inertial>
   </link>
@@ -102,4 +112,9 @@
     <origin xyz="${-wheelbase/2} ${-track/2} ${wheel_vertical_offset}" rpy="0 0 0" />
   </xacro:tugbot_wheel>
+  <xacro:include filename="$(find velodyne_description)/urdf/VLP-16.urdf.xacro"/>
+  <VLP-16 parent="base_link" name="velodyne" topic="/velodyne_points">
+      <!-- The 0.2 will most likely have to be adjusted to fit -->
+      <origin xyz="0 0 0.1" rpy="0 0 0" />
+  </VLP-16>
   <gazebo>
     <plugin name="gazebo_ros_control" filename="libgazebo_ros_control.so">

Commit message: Added standalone urdf viewing:

File: tugbot_description/urdf/tugbot.urdf.xacro (robot description, xacro)
@@ -2,4 +2,5 @@
 <robot name="tugbot" xmlns:xacro="http://ros.org/wiki/xacro">
   <xacro:arg name="robot_namespace" default="/" />
+  <xacro:arg name="vlp16_enabled" default="false" />
   <xacro:property name="M_PI" value="3.14159"/>
   <xacro:macro name="tugbot_wheel" params="wheel_prefix left_wheel *joint_pose">
@@ -112,9 +113,11 @@
     <origin xyz="${-wheelbase/2} ${-track/2} ${wheel_vertical_offset}" rpy="0 0 0" />
   </xacro:tugbot_wheel>
-  <xacro:include filename="$(find velodyne_description)/urdf/VLP-16.urdf.xacro"/>
-  <VLP-16 parent="base_link" name="velodyne" topic="/velodyne_points">
-      <!-- The 0.2 will most likely have to be adjusted to fit -->
-      <origin xyz="0 0 0.1" rpy="0 0 0" />
-  </VLP-16>
+  <xacro:if value="$(arg vlp16_enabled)">
+    <xacro:include filename="$(find velodyne_description)/urdf/VLP-16.urdf.xacro"/>
+    <VLP-16 parent="base_link" name="velodyne" topic="/velodyne_points">
+        <!-- The 0.2 will most likely have to be adjusted to fit -->
+        <origin xyz="0 0 0.1" rpy="0 0 0" />
+    </VLP-16>
+  </xacro:if>
   <gazebo>
     <plugin name="gazebo_ros_control" filename="libgazebo_ros_control.so">
